Commit message: add camera

File: denso_robot_descriptions/vs060_description/vs060.urdf (robot description, URDF)
Before this commit: robot vs060, 8 links, 7 joints
Links:
- added link camera_link, mass 1e-5; collision box size=0.1 0.07 0.05; visual box size=0.1 0.07 0.05
- added link camera_link_optical
Joints:
- added joint camera_joint: type fixed, parent J6, child camera_link, origin xyz=0 0 0.15 rpy=0 -1.5708 0, axis 1 0 0
- added joint camera_optical_joint: type fixed, parent camera_link, child camera_link_optical, origin xyz=0 0 0 rpy=-1.5708 0 -1.5708

Commit message: add pattern

File: denso_robot_descriptions/vs060_description/vs060.urdf (robot description, URDF)
Before this commit: robot vs060, 10 links, 9 joints
Links:
- added link pattern, mass 1; collision box size=0.22 0.18 0.002; visual mesh filename=package://denso_robot_descriptions/vs060_description/test2.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 scale=1 1 1
Joints:
- added joint joint_pattern: type fixed, parent world, child pattern, origin xyz=1.700000 1.000000 0.03 rpy=0.000000 0.000000 0.000000

Commit message: add image saver and calibration flow

File: denso_robot_descriptions/vs060_description/vs060.urdf (robot description, URDF)
Before this commit: robot vs060, 11 links, 10 joints
Links:
- link camera_link: geometry collision box size=0.075 0.060 0.030; visual box size=0.075 0.060 0.030
- link pattern: geometry collision box size=0.22 0.18 0.002; visual mesh filename=package://denso_robot_descriptions/vs060_description/patter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 scale=1 1 1
Joints:
- joint camera_joint: origin xyz=0 0 0.15 rpy=0 -1.5708 0 -> xyz=0 0 0.05 rpy=0 -1.5708 0
- joint joint_pattern: origin xyz=1.700000 1.000000 0.03 rpy=0.000000 0.000000 0.000000 -> xyz=0.500000 0.000000 0.001 rpy=0.000000 0.000000 0.000000

Commit message: add camera trigger

File: denso_robot_descriptions/vs060_description/vs060.urdf (robot description, URDF)
Before this commit: robot vs060, 11 links, 10 joints
Joints:
- joint camera_joint: origin xyz=0 0 0.05 rpy=0 -1.5708 0 -> xyz=0 0 0.05 rpy=0 -1.5707963 0
- joint camera_optical_joint: origin xyz=0 0 0 rpy=-1.5708 0 -1.5708 -> xyz=0 0 0 rpy=-1.5707963 0 -1.5707963
- joint joint_pattern: origin xyz=0.500000 0.000000 0.001 rpy=0.000000 0.000000 0.000000 -> xyz=0.500000 0.000000 0.001 rpy=0.000000 0.000000 1.5707963

Commit message: Add robot control, mongoDB and modify the description file for vs6242 robot, Now it can control the real denso robot!

File: denso_robot_descriptions/vs060_description/vs060.urdf (robot description, URDF)
Before this commit: robot vs060, 11 links, 10 joints
Joints:
- joint joint_pattern: origin xyz=0.500000 0.000000 0.001 rpy=0.000000 0.000000 1.5707963 -> xyz=0.300000 0.000000 0.001 rpy=0.000000 0.000000 1.5707963
