Commit message: add Readme

File: denso_robot_descriptions/vs6242_description/vs6242.urdf (robot description, URDF)
Before this commit: robot vs6242, 8 links, 7 joints
Links:
- added link camera_link, mass 1e-5; collision box size=0.075 0.060 0.030; visual box size=0.075 0.060 0.030
- added link camera_link_optical
- added link pattern, mass 1; collision box size=0.22 0.18 0.002; visual mesh filename=package://denso_robot_descriptions/vs060_description/patter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 scale=1 1 1
Joints:
- added joint camera_joint: type fixed, parent J6, child camera_link, origin xyz=0 0 0.05 rpy=0 -1.5707963 0, axis 1 0 0
- added joint camera_optical_joint: type fixed, parent camera_link, child camera_link_optical, origin xyz=0 0 0 rpy=-1.5707963 0 -1.5707963
- added joint joint_pattern: type fixed, parent world, child pattern, origin xyz=0.300000 0.000000 0.001 rpy=0.000000 0.000000 1.5707963

Commit message: hole searching

File: denso_robot_descriptions/vs6242_description/vs6242.urdf (robot description, URDF)
Before this commit: robot vs6242, 11 links, 10 joints
Links:
- added link marker, mass 1; collision box size=0.03 0.03 0.002; visual mesh filename=package://denso_robot_descriptions/vs6242_description/diamo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 scale=1 1 1
- added link pcb; visual mesh filename=package://denso_robot_descriptions/vs6242_description/pcb.d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 scale=0.4 0.4 0.4
- link pattern: geometry collision box size=0.22 0.18 0.002; visual mesh filename=package://denso_robot_descriptions/vs6242_description/patte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 scale=1 1 1
Joints:
- added joint joint_marker: type fixed, parent pcb, child marker, origin xyz=0.05000 0.060000 0.01 rpy=0.000000 0.000000 1.5707963
- added joint joint_pcb: type fixed, parent world, child pcb, origin xyz=0.000000 -0.350000 0.001 rpy=0.000000 0.000000 1.5707963

Commit message: hole searching

File: denso_robot_descriptions/vs6242_description/vs6242.urdf (robot description, URDF)
Before this commit: robot vs6242, 13 links, 12 joints
Links:
- link pcb: mass None -> 1; geometry collision box size=0.03 0.03 0.002; visual mesh filename=package://denso_robot_descriptions/vs6242_description/pcb.d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 scale=0.4 0.4 0.4
Joints:
- joint joint_marker: origin xyz=0.05000 0.060000 0.01 rpy=0.000000 0.000000 1.5707963 -> xyz=-0.06000 -0.30000 0.011 rpy=0.000000 0.000000 1.5707963; parent pcb -> world

Commit message: ac and af is perfect , NEXT: solveXZ have to improve

File: denso_robot_descriptions/vs6242_description/vs6242.urdf (robot description, URDF)
Before this commit: robot vs6242, 13 links, 12 joints
Joints:
- joint camera_joint: origin xyz=0 0 0.05 rpy=0 -1.5707963 0 -> xyz=-0.035 0 0.05 rpy=0 -1.5707963 0
- joint joint_pattern: origin xyz=0.300000 0.000000 0.001 rpy=0.000000 0.000000 1.5707963 -> xyz=0.310000 0.050000 0.001 rpy=0.00000 0.000000 -1.047197551

Commit message: insert ok
ZXzxczxc

File: denso_robot_descriptions/vs6242_description/vs6242.urdf (robot description, URDF)
Before this commit: robot vs6242, 13 links, 12 joints
Joints:
- joint camera_joint: origin xyz=-0.035 0 0.05 rpy=0 -1.5707963 0 -> xyz=-0.040 0 0.040 rpy=0 -1.5707963 0
- joint joint_marker: origin xyz=-0.06000 -0.30000 0.011 rpy=0.000000 0.000000 1.5707963 -> xyz=-0.06000 -0.30000 0.010 rpy=0.000000 0.000000 1.5707963
- joint joint_pattern: origin xyz=0.310000 0.050000 0.001 rpy=0.00000 0.000000 -1.047197551 -> xyz=0.300000 0.000000 0.001 rpy=0.000000 0.000000 -1.5707963267948966
